File: _autosave-FMCW_0.kicad_pcb (KiCad board)
At the start: 6 copper layers, 100 x 100 mm, 311 parts, among them J1 Conn_02x07_Odd_Even, J2 HFJ11-1G41E-L12RL, J3 Conn_Coaxial_Small, J4 USB_C_Receptacle_USB2.0_16P, J5 Barrel_Jack_Switch, J6 USB_C_Receptacle_USB2.0_16P, J7 Conn_Coaxial_Small, J8 Conn_Coaxial_Small, SW1 SW_SPDT, SW2 SW_Push, SW3 SW_DIP_x04, SW4 SW_Push, U1 PAT1220-C-6DB, U10 LMX2491, U11 MAX275X, U12 5400BL15B050, U13 5400BL15B050, U14 ADL5380, U15 TPS259620, U16 Kria K24 SoM, U17 AP2127K-1.0, U18 AP2127K-2.5, U19 DP83867CRRGZR, U2 PAT1220-C-6DB, U20 SN74LVC2G06, U21 TPS53119, U22 TPS54308, U23 TPS54308, U24 CSD87352Q5D, U25 SN74LVC1G06, U26 TPS3839K33DBZR, U27 TPS3839G18DBZR, U28 AP22816AKEWT, U29 USB3300-EZK, U3 LMK1C1103A, U30 FT231XQ, U4 AP63200WU, U5 TLV76750QWDRBxQ1, U6 TLV76733QWDRBxQ1, U7 TPS3839K50DBZR, U8 TPS3839K33DBZR, U9 MCP3911, Y1 ECS-2520MV-160-BN, Y2 25MHz, Y3 ECS-240-12-37B-CKY-TR

Commit message: finished routing (i think)
Routing:
- net /RFFE/ADC/adc_dvdd: track 3.58 -> 10.2 mm
- net +3.3VA: track 13.1 -> 16.0 mm, vias 6 -> 9
- net Net-(U14-ENBL): track 0.00 -> 1.91 mm
- net Net-(C39-Pad1): track 0.00 -> 1.28 mm
- net Net-(C38-Pad1): track 0.00 -> 1.28 mm
- net Net-(U14-LOIN): track 0.00 -> 1.24 mm
- net Net-(U14-LOIP): track 0.00 -> 1.24 mm
Changed lines of the file:
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@@
 	)
 	(segment
+		(start 112.3696 48.6716)
+		(end 112.3888 48.6908)
+		(width 0.2032)
+		(layer "F.Cu")
+		(net "+3.3VA")
+	)
+	(segment
 		(start 109.6335 56.3523)
 		(end 109.6335 57.0277)
@@
 	)
 	(segment
+		(start 92.71 61.8764)
+		(end 93.3164 61.8764)
+		(width 0.254)
+		(layer "F.Cu")
+		(net "+3.3VA")
+	)
+	(segment
 		(start 111.7412 54.8523)
 		(end 111.76 54.8711)
@@
 	)
 	(segment
+		(start 112.3696 43.6495)
+		(end 112.9355 43.6495)
+		(width 0.2032)
+		(layer "F.Cu")
+		(net "+3.3VA")
+	)
+	(segment
+		(start 112.3696 48.1147)
+		(end 112.3696 48.6716)
+		(width 0.2032)
+		(layer "F.Cu")
+		(net "+3.3VA")
+	)
+	(segment
 		(start 110.019 57.0398)
 		(end 110.0266 57.0474)
@@
 	)
 	(segment
+		(start 93.3164 61.8764)
+		(end 93.3388 61.8988)
+		(width 0.254)
+		(layer "F.Cu")
+		(net "+3.3VA")
+	)
+	(segment
 		(start 109.6335 54.8523)
 		(end 111.7412 54.8523)
@@
 	)
 	(segment
+		(start 112.9355 43.6495)
+		(end 112.9984 43.7124)
+		(width 0.2032)
+		(layer "F.Cu")
+		(net "+3.3VA")
+	)
+	(segment
 		(start 108.946 57.0398)
 		(end 109.6456 57.0398)
@@
 	)
 	(segment
+		(start 91.7448 61.8764)
+		(end 92.71 61.8764)
+		(width 0.254)
+		(layer "F.Cu")
+		(net "+3.3VA")
+	)
+	(segment
 		(start 109.6335 57.0277)
 		(end 109.6456 57.0398)
@@
 	)
 	(via
+		(at 93.3388 61.8988)
+		(size 0.508)
+		(drill 0.3048)
+		(layers "F.Cu" "B.Cu")
+		(net "+3.3VA")
+	)
+	(via
+		(at 112.3888 48.6908)
+		(size 0.508)
+		(drill 0.3048)
+		(layers "F.Cu" "B.Cu")
+		(net "+3.3VA")
+	)
+	(via
 		(at 120.1104 53.2628)
 		(size 0.8128)
@@
 	)
 	(via
+		(at 112.9984 43.7124)
+		(size 0.508)
+		(drill 0.3048)
+		(layers "F.Cu" "B.Cu")
+		(net "+3.3VA")
+	)
+	(via
 		(at 111.3982 57.8094)
 		(size 0.508)
@@
 	)
 	(segment
+		(start 85.6863 51.5681)
+		(end 84.6836 52.5708)
+		(width 0.254)
+		(layer "F.Cu")
+		(net "Net-(U14-ENBL)")
+	)
+	(segment
+		(start 84.6836 52.5708)
+		(end 84.6836 52.8808)
+		(width 0.254)
+		(layer "F.Cu")
+		(net "Net-(U14-ENBL)")
+	)
+	(segment
+		(start 85.8658 51.5681)
+		(end 85.6863 51.5681)
+		(width 0.254)
+		(layer "F.Cu")
+		(net "Net-(U14-ENBL)")
+	)
+	(segment
+		(start 86.8658 51.5681)
+		(end 86.8658 52.5522)
+		(width 0.254)
+		(layer "F.Cu")
+		(net "Net-(U14-LOIP)")
+	)
+	(segment
+		(start 86.8658 52.5522)
+		(end 86.6876 52.7304)
+		(width 0.254)
+		(layer "F.Cu")
+		(net "Net-(U14-LOIP)")
+	)
+	(segment
+		(start 87.3658 51.5681)
+		(end 87.3658 52.5398)
+		(width 0.254)
+		(layer "F.Cu")
+		(net "Net-(U14-LOIN)")
+	)
+	(segment
+		(start 87.3658 52.5398)
+		(end 87.5564 52.7304)
+		(width 0.254)
+		(layer "F.Cu")
+		(net "Net-(U14-LOIN)")
+	)
+	(segment
 		(start 89.0595 49.8816)
 		(end 91.9134 49.8816)
@@
 	)
 	(segment
+		(start 88.5164 52.7304)
+		(end 88.5164 53.3132)
+		(width 0.254)
+		(layer "F.Cu")
+		(net "Net-(C38-Pad1)")
+	)
+	(segment
+		(start 88.5164 53.3132)
+		(end 88.022 53.8076)
+		(width 0.254)
+		(layer "F.Cu")
+		(net "Net-(C38-Pad1)")
+	)
+	(segment
+		(start 85.7276 52.7304)
+		(end 85.7276 53.3132)
+		(width 0.254)
+		(layer "F.Cu")
+		(net "Net-(C39-Pad1)")
+	)
+	(segment
+		(start 85.7276 53.3132)
+		(end 86.222 53.8076)
+		(width 0.254)
+		(layer "F.Cu")
+		(net "Net-(C39-Pad1)")
+	)
+	(segment
 		(start 147.3745 78.3881)
 		(end 147.3745 81.0937)
@@
 	)
 	(segment
+		(start 90.142 60.8864)
+		(end 88.3604 62.668)
+		(width 0.508)
+		(layer "In3.Cu")
+		(net "/RFFE/ADC/adc_dvdd")
+	)
+	(segment
+		(start 88.3604 64.642)
+		(end 86.8618 66.1406)
+		(width 0.508)
+		(layer "In3.Cu")
+		(net "/RFFE/ADC/adc_dvdd")
+	)
+	(segment
+		(start 88.3604 62.668)
+		(end 88.3604 64.642)
+		(width 0.508)
+		(layer "In3.Cu")
+		(net "/RFFE/ADC/adc_dvdd")
+	)
+	(segment
 		(start 133.7564 114.9284)
 		(end 133.3688 115.316)
@@
 		(polygon
 			(pts
-				(xy 120.72 50.799) (xy 98.114 50.799) (xy 96.082 52.831) (xy 75 52.831) (xy 75 67.69) (xy 89.605 67.69)
-				(xy 94.558 62.737) (xy 120.72 62.737)
+				(xy 120.72 50.8244) (xy 118.7896 50.8244) (xy 114.624 46.6588) (xy 114.624 44.4236) (xy 113.4556 43.2552)
+				(xy 105.734 43.2552) (xy 96.1328 52.8564) (xy 75 52.8564) (xy 75 67.69) (xy 89.605 67.69) (xy 94.558 62.737)
+				(xy 120.72 62.737)
 			)
 		)
@@
 		(polygon
 			(pts
-				(xy 120.72 35.051) (xy 120.72 50.545) (xy 98.071594 50.543318) (xy 97.987 50.545) (xy 95.955 52.577)
-				(xy 75 52.577) (xy 75 35.051)
+				(xy 120.72 35.051) (xy 120.72 50.57055) (xy 118.942084 50.570484) (xy 114.9288 46.5572) (xy 114.9288 44.322)
+				(xy 113.608 43.0012) (xy 105.5308 43.0012) (xy 95.955 52.577) (xy 75 52.577) (xy 75 35.051)
 			)
 		)
