File: FMCW_0.kicad_sch (KiCad schematic)
At the start: 8 parts, among them J3 Conn_Coaxial_Small, J5 Barrel_Jack_Switch, J7 Conn_Coaxial_Small, J8 Conn_Coaxial_Small

Commit message: finished routing (i think)
Parts:
- added H5, H6: MountingHole_Pad, MountingHole:MountingHole_3.2mm_M3_DIN965_Pad, symbol Mechanical:MountingHole_Pad
Connections:
- net GND: now also H5.1, H6.1
Other:
- moved on the sheet: H1, H2, H3, H4

Commit message: Imon Schematic and DRC checking changes -Added current monitor ADC for Imon -Fixed unconnected nets -Added shorting resistor between both output power on signals from Kria SoM
Other:
- sheet fpga ports: added Imon; removed none
Changed lines of the file:
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@@
+	(wire
+		(pts
+			(xy 105.41 57.15) (xy 97.79 57.15)
+		)
+		(stroke
+			(width 0)
+			(type default)
+		)
+	)
 	(wire
 		(pts
@@
 	(wire
 		(pts
+			(xy 114.3 90.17) (xy 105.41 90.17)
+		)
+		(stroke
+			(width 0)
+			(type default)
+		)
+	)
+	(wire
+		(pts
 			(xy 251.46 53.34) (xy 251.46 58.42)
 		)
@@
 		(pts
 			(xy 251.46 58.42) (xy 251.46 66.04)
+		)
+		(stroke
+			(width 0)
+			(type default)
+		)
+	)
+	(wire
+		(pts
+			(xy 105.41 90.17) (xy 105.41 57.15)
 		)
 		(stroke
@@
 			)
 		)
+		(pin "Imon" input
+			(at 114.3 90.17 180)
+			(effects
+				(font
+					(size 1.27 1.27)
+				)
+				(justify left)
+			)
+		)
