File: fpga.kicad_sch (KiCad schematic)
At the start: 0 parts

Commit message: Imon Schematic and DRC checking changes -Added current monitor ADC for Imon -Fixed unconnected nets -Added shorting resistor between both output power on signals from Kria SoM
Other:
- sheet fpga_ja ports: added Imon; removed none
Changed lines of the file:
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@@
+	(wire
+		(pts
+			(xy 83.82 77.47) (xy 101.6 77.47)
+		)
+		(stroke
+			(width 0)
+			(type default)
+		)
+	)
 	(wire
 		(pts
@@
 		(shape input)
 		(at 83.82 49.53 180)
+		(effects
+			(font
+				(size 1.27 1.27)
+			)
+			(justify right)
+		)
+	)
+	(hierarchical_label "Imon"
+		(shape input)
+		(at 83.82 77.47 180)
 		(effects
 			(font
@@
 			)
 		)
+		(pin "Imon" input
+			(at 101.6 77.47 180)
+			(effects
+				(font
+					(size 1.27 1.27)
+				)
+				(justify left)
+			)
+		)
