File: FMCW_0.kicad_pcb (KiCad board)
At the start: 6 copper layers, 100 x 100 mm, 321 parts, among them J1 Conn_02x07_Odd_Even, J2 HFJ11-1G41E-L12RL, J3 Conn_Coaxial_Small, J4 USB_C_Receptacle_USB2.0_16P, J5 Barrel_Jack_Switch, J6 USB_C_Receptacle_USB2.0_16P, J7 Conn_Coaxial_Small, J8 Conn_Coaxial_Small, SW1 SW_SPDT, SW2 SW_Push, SW3 SW_DIP_x04, SW4 SW_Push, U1 PAT1220-C-6DB, U10 LMX2491, U11 MAX275X, U12 5400BL15B050, U13 5400BL15B050, U14 ADL5380, U15 TPS259620, U16 Kria K24 SoM, U17 AP2127K-1.0, U18 AP2127K-2.5, U19 DP83867CRRGZR, U2 PAT1220-C-6DB, U20 SN74LVC2G06, U21 TPS53119, U22 TPS54308, U23 TPS54308, U24 CSD87352Q5D, U25 SN74LVC1G06, U26 TPS3839K33DBZR, U27 TPS3839G18DBZR, U28 AP22816AKEWT, U29 USB3300-EZK, U3 LMK1C1103A, U30 FT231XQ, U31 MCP3221, U4 AP63200WU, U5 TLV76750QWDRBxQ1, U6 TLV76733QWDRBxQ1, U7 TPS3839K50DBZR, U8 TPS3839K33DBZR, U9 MCP3911, Y1 ECS-2520MV-160-BN, Y2 25MHz, Y3 ECS-240-12-37B-CKY-TR

Commit message: Schematic and layout updates:
-Removed some extraneous wires on schematic sheets. May be some more.
-Length matched RGMII and ULPI. Maybe need to look at TFT.
-Updated some digikey part numbers.
-Added some extra file nonesense to .gitignore
Routing:
- net /fpga/eth/e_tx_ctrl: track 32.2 -> 63.8 mm
- net /fpga/eth/e_tx_clk: track 31.5 -> 60.4 mm
- net /fpga/eth/e_tx_d1: track 31.3 -> 58.5 mm
- net /fpga/eth/e_rx_ctrl: track 32.9 -> 59.7 mm
- net /fpga/eth/e_tx_d2: track 31.3 -> 57.6 mm
- net /fpga/eth/e_rx_d3: track 31.3 -> 52.8 mm
- net /fpga/eth/e_rx_clk: track 31.1 -> 51.0 mm
- net /fpga/eth/e_rx_d0: track 31.1 -> 48.5 mm
- net /fpga/usb_host/u_d1: track 64.7 -> 77.6 mm
- net /fpga/usb_host/u_clkout: track 67.9 -> 77.2 mm
- net /fpga/usb_host/u_d2: track 64.6 -> 73.9 mm
- net /fpga/usb_host/u_d3: track 64.7 -> 71.9 mm
- net /fpga/usb_host/u_d0: track 64.6 -> 69.3 mm
- net /fpga/usb_host/u_d6: track 64.4 -> 69.0 mm
- net /fpga/eth/eth_rx_clk: track 6.75 -> 9.95 mm
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