File: eth.kicad_sch (KiCad schematic)
At the start: 41 parts, among them J2 HFJ11-1G41E-L12RL, U17 AP2127K-1.0, U18 AP2127K-2.5, U19 DP83867CRRGZR, U20 SN74LVC2G06, Y2 25MHz

Commit message: Schematic and layout updates:
-Removed some extraneous wires on schematic sheets. May be some more.
-Length matched RGMII and ULPI. Maybe need to look at TFT.
-Updated some digikey part numbers.
-Added some extra file nonesense to .gitignore
Parts:
- C59, C60, C61, C62, C68, C69, C70, C74, C75, C76, C79, C82: Digikey PN (none) -> 1276-1067-1-ND
- C65, C66, C67, C71, C72, C73, C77, C78, C80, C81: Digikey PN (none) -> 1276-1043-1-ND
- R53: Digikey PN (none) -> P1.50KLCT-ND
- R55, R56: Digikey PN (none) -> 311-220LRCT-ND
