File: fpga_pin.kicad_sch (KiCad schematic)
At the start: 60 parts, among them SW4 SW_Push, U21 TPS53119, U22 TPS54308, U23 TPS54308, U24 CSD87352Q5D, U25 SN74LVC1G06, U26 TPS3839K33DBZR, U27 TPS3839G18DBZR

Commit message: some changes. layout routing done. need to check eth/usb length matching
Parts:
- U21: footprint Package_DFN_QFN:VQFN-16-1EP_3x3mm_P0.5mm_EP1.45x1.45mm_ThermalVias -> Package_DFN_QFN:VQFN-16-1EP_3x3mm_P0.5mm_EP1.45x1.45mm
Changed lines of the file:
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@@
 			)
 		)
-		(property "Footprint" "Package_DFN_QFN:VQFN-16-1EP_3x3mm_P0.5mm_EP1.45x1.45mm_ThermalVias"
+		(property "Footprint" "Package_DFN_QFN:VQFN-16-1EP_3x3mm_P0.5mm_EP1.45x1.45mm"
 			(at 91.44 31.75 0)
 			(hide yes)

Commit message: Schematic and layout updates:
-Removed some extraneous wires on schematic sheets. May be some more.
-Length matched RGMII and ULPI. Maybe need to look at TFT.
-Updated some digikey part numbers.
-Added some extra file nonesense to .gitignore
Parts:
- C100, C101, C107, C91, C92, C93, C94, C99: Digikey PN (none) -> 1276-1043-1-ND
- C103: Digikey PN (none) -> 587-3466-1-ND
- C104, C105, C106, C108, C109: Digikey PN (none) -> 587-5466-1-ND
- C87: Digikey PN (none) -> 1276-1067-1-ND
- C89, C90: Digikey PN (none) -> 490-7202-1-ND
- R59, R69, R76: Digikey PN (none) -> RMCF0402FT10K0CT-ND
- R60, R65, R74: Digikey PN (none) -> 541-22.0LCT-ND
- R64: Digikey PN (none) -> 311-1.00KLRCT-ND
- R94: Digikey PN (none) -> 311-470LRCT-ND
