File: rffe_ps.kicad_sch (KiCad schematic)
At the start: 22 parts, among them U4 AP63200WU, U5 TLV76750QWDRBxQ1, U6 TLV76733QWDRBxQ1, U7 TPS3839K50DBZR, U8 TPS3839K33DBZR

Commit message: Schematic and layout updates:
-Removed some extraneous wires on schematic sheets. May be some more.
-Length matched RGMII and ULPI. Maybe need to look at TFT.
-Updated some digikey part numbers.
-Added some extra file nonesense to .gitignore
Parts:
- C11, C12: Digikey PN (none) -> 1276-1043-1-ND
Changed lines of the file:
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@@
+			)
+		)
+		(property "Digikey PN" "1276-1043-1-ND"
+			(at 231.14 121.92 0)
+			(hide yes)
+			(show_name no)
+			(do_not_autoplace no)
+			(effects
+				(font
+					(size 1.27 1.27)
+				)
 			)
 		)
@@
 			(at 231.14 82.55 0)
 			(hide yes)
+			(show_name no)
+			(do_not_autoplace no)
+			(effects
+				(font
+					(size 1.27 1.27)
+				)
+			)
+		)
+		(property "Digikey PN" "1276-1043-1-ND"
+			(at 231.14 82.55 0)
+			(hide yes)
