File: usb_host.kicad_sch (KiCad schematic)
At the start: 37 parts, among them J6 USB_C_Receptacle_USB2.0_16P, U28 AP22816AKEWT, U29 USB3300-EZK, Y3 ECS-240-12-37B-CKY-TR

Commit message: Schematic and layout updates:
-Removed some extraneous wires on schematic sheets. May be some more.
-Length matched RGMII and ULPI. Maybe need to look at TFT.
-Updated some digikey part numbers.
-Added some extra file nonesense to .gitignore
Parts:
- R79: Digikey PN 311-20.0KLRCT-ND -> 311-1.00KLRCT-ND
- R98: Digikey PN 311-820LRCT-ND -> (none)
Changed lines of the file:
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@@
 			)
 		)
-		(property "Digikey PN" "311-20.0KLRCT-ND"
+		(property "Digikey PN" "311-1.00KLRCT-ND"
 			(at 93.98 33.02 0)
 			(hide yes)
@@
 			)
 		)
-		(property "Digikey PN" "311-820LRCT-ND"
+		(property "Digikey PN" ""
 			(at 106.68 116.84 0)
 			(hide yes)
